Commit message: Navigation, optic flow and robot description

File: urdf_tinker/tinker.urdf (robot description, URDF)
Before this commit: robot tinker, 17 links, 16 joints
Links:
- removed link laser_scan_sensor_link
- added link laser; visual cylinder length=0.05 radius=0.025
Joints:
- joint base_link_to_arm_holder: origin xyz=0 0 0.3 rpy=0 0 0 -> xyz=0 0 0.3 rpy=0 0 -1.57
- joint base_to_chassis: origin xyz=0 -0.1 -0.45 -> xyz=0 -0.1 -0.45 rpy=0 0 -1.57
- joint camera_holder_to_laser_scan_sensor: child laser_scan_sensor_link -> laser

Commit message: regular commit

File: urdf_tinker/tinker.urdf (robot description, URDF)
Before this commit: robot tinker, 17 links, 16 joints
Joints:
- joint base_to_chassis: origin xyz=0 -0.1 -0.45 rpy=0 0 -1.57 -> xyz=-0.0707 0 -0.45 rpy=0 0 -1.57
