Commit message: regular push

File: tinker_2dnav/tinker.urdf (robot description, URDF)
Before this commit: robot tinker, 17 links, 16 joints
Links:
- added link laser_bottom; visual cylinder length=0.05 radius=0.025
- added link laser_bottom_holder; visual box size=0.10 .20 .01
- added link robot_base; visual cylinder length=1.2 radius=0.08
- link base_link: geometry 
Joints:
- removed joint base_link_to_arm_holder
- removed joint base_link_to_camera
- added joint base_link_to_base: type fixed, parent base_link, child robot_base, origin xyz=0 0 0.6 rpy=0 0 0
- added joint chasis_to_laser_bottom_holder: type fixed, parent chassis, child laser_bottom_holder, origin xyz=0 0.25 0 rpy=0 0 0 
- added joint laser_bottom_holder_to_laser_bottom: type fixed, parent laser_bottom_holder, child laser_bottom, origin xyz=0 0 -0.05 rpy=0 3.14 -1.57
- added joint robot_base_to_arm_holder: type prismatic, parent robot_base, child arm_holder, origin xyz=0 0 0.3 rpy=0 0 -1.57, axis 0 0 1, limit lower=-0.1 upper=0.1 effort=30 velocity=1.0
- added joint robot_base_to_camera: type fixed, parent robot_base, child camera_holder, origin xyz=0 0 0.65 rpy=0 0 0.7853
- joint base_to_chassis: origin xyz=0 -0.1 -0.45 rpy=0 0 -1.57 -> xyz=-0.0707  0 -0.45 rpy=0 0 -1.57; parent base_link -> robot_base

File: urdf_tinker/tinker.urdf (robot description, URDF)
Before this commit: robot tinker, 17 links, 16 joints
Links:
- added link laser_bottom; visual cylinder length=0.05 radius=0.025
- added link laser_bottom_holder; visual box size=0.10 .20 .01
- added link robot_base; visual cylinder length=1.2 radius=0.08
- link base_link: geometry 
Joints:
- removed joint base_link_to_arm_holder
- removed joint base_link_to_camera
- added joint base_link_to_base: type fixed, parent base_link, child robot_base, origin xyz=0 0 0.6 rpy=0 0 0
- added joint chasis_to_laser_bottom_holder: type fixed, parent chassis, child laser_bottom_holder, origin xyz=0 0.25 0 rpy=0 0 0 
- added joint laser_bottom_holder_to_laser_bottom: type fixed, parent laser_bottom_holder, child laser_bottom, origin xyz=0 0 -0.05 rpy=0 3.14 0
- added joint robot_base_to_arm_holder: type prismatic, parent robot_base, child arm_holder, origin xyz=0 0 0.3 rpy=0 0 -1.57, axis 0 0 1, limit lower=-0.1 upper=0.1 effort=30 velocity=1.0
- added joint robot_base_to_camera: type fixed, parent robot_base, child camera_holder, origin xyz=0 0 0.65 rpy=0 0 0.7853
- joint base_to_chassis: origin xyz=-0.0707 0 -0.45 rpy=0 0 -1.57 -> xyz=-0.0707  0 -0.45 rpy=0 0 -1.57; parent base_link -> robot_base
